File: ProjectKiCADSchematic/ProjectKiCADSchematic.kicad_sch (KiCad schematic)
At the start: 0 parts

Commit message: just a few commants
Parts:
- added A1: RaspberryPi_Pico_W, Module:RaspberryPi_Pico_W_SMD_HandSolder, symbol MCU_Module:RaspberryPi_Pico_W
- added A2: RaspberryPi_Pico_W_Debug, Module:RaspberryPi_Pico_SMD_HandSolder, symbol MCU_Module:RaspberryPi_Pico_Debug
- added B1: Vibration motor right, VZ43FM1B8230001L:XDCR_VZ43FM1B8230001L, symbol VZ43FM1B8230001L:VZ43FM1B8230001L
- added B2: Vibration motor left, VZ43FM1B8230001L:XDCR_VZ43FM1B8230001L, symbol VZ43FM1B8230001L:VZ43FM1B8230001L
- added BZ1: Buzzer, symbol Device:Buzzer
- added D1, D2: 1N4148, Diode_THT:D_DO-35_SOD27_P7.62mm_Horizontal, symbol Diode:1N4148
- added Q1, Q2: 2N2222, 2N2222:TO127P584H533-3, symbol 2N2222:2N2222
- added U1, U2: HC-SR04, distanse sensore right, symbol HC-SR04:HC-SR04
Connections:
- new net: A2.21 (GPIO16), U1.2 (TRIG)
- new net: A2.22 (GPIO17), U1.3 (ECHO)
- new net: B1.2, D1.1 (K)
- new net: A1.7 (GPIO5), A2.1 (GPIO0)
- new net: A2.19 (GPIO14), U2.3 (ECHO)
- new net: A1.6 (GPIO4), A2.2 (GPIO1)
- new net: A2.20 (GPIO15), U2.2 (TRIG)
- new net: A2.24 (GPIO18), BZ1.2 (-)
- new net: A2.25 (GPIO19), Q1.2
- new net: A2.26 (GPIO20), Q2.2
- new net: A1.4 (GPIO2), A2.D1 (SWCLK)
- new net: A1.5 (GPIO3), A2.D3 (SWDIO)
- new net: B1.1, Q2.3
- new net: B2.2, D2.1 (K)
- new net: B2.1, Q1.3
- new net +3.3V: A1.13 (GND), A1.18 (GND), A1.23 (GND), A1.28 (GND), A1.3 (GND), A1.38 (GND), A1.39 (VSYS), A1.8 (GND), A2.13 (GND), A2.18 (GND), A2.23 (GND), A2.28 (GND), A2.3 (GND), A2.38 (GND), A2.39 (VSYS), A2.8 (GND), A2.D2 (GND), BZ1.1 (+), D1.2 (A), D2.2 (A), Q1.1, Q2.1, U1.1 (VCC), U1.4 (GND), U2.1 (VCC), U2.4 (GND)
